Commit message: lab3_TODO_kin

File: manipulator/urdf/base_and_limits.xacro (robot description, xacro)
@@ -8,12 +8,15 @@
     <xacro:property name="base_height"      value="0.1"     />
     <xacro:property name="base_height_half" value="${base_height/2.0}" />
+    <xacro:property name="gripper_size"        value="0.4 0.4" />
+    <xacro:property name="gripper_height"      value="0.4"     />
+    <xacro:property name="gripper_height_half" value="${gripper_height/2.0}" />
+    <xacro:property name="gripper_limit_lower"      value="-0.4"  />
+    <xacro:property name="gripper_limit_upper"      value="0.4"   />
     <xacro:property name="l00"          value="base_link"           />
 	<xacro:property name="l01"          value="link_01"             />
 	<xacro:property name="l02"          value="link_02"             />
 	<xacro:property name="l03"          value="link_03"             />
-	<xacro:property name="l04"          value="link_04"             />
 	<xacro:property name="R01"          value="0.25"             />
 	<xacro:property name="R02"          value="0.2"             />
 	<xacro:property name="R03"          value="0.15"             />
-	<xacro:property name="R04"          value="0.1"             />
 </robot>

File: manipulator/urdf/dh_parameters.xacro (robot description, xacro)
@@ -6,23 +6,16 @@
 	<xacro:property name="L1"    	value="0.0"	/>
 	<xacro:property name="phi1"    	value="0.0"	/>
-	<xacro:property name="a1"    	value="0"	/>
-	<xacro:property name="alpha1"	value="${pi/2.0}"	/>
+	<xacro:property name="type0"    	value="revolute"	/>
+	<xacro:property name="a1"    	value="1"	/>
+	<xacro:property name="alpha1"	value="${0}"	/>
 	<xacro:property name="d2"    	value="2"	/>
-	<xacro:property name="L2"    	value="2.0"	/>
-	<xacro:property name="phi2"    	value="0.0"	/>
-	<xacro:property name="a2"    	value="0"	/>
-	<xacro:property name="alpha2"	value="${pi/2.0}"	/>
-	<xacro:property name="d3"    	value="1.5"	/>
-	<xacro:property name="L3"    	value="1.5"	/>
-	<xacro:property name="phi3"    	value="0.0"	/>
-	<xacro:property name="a3"    	value="1"	/>
-	<xacro:property name="alpha3"	value="${0}"	/>
-	<xacro:property name="d4"    	value="1"	/>
-	<xacro:property name="L4"    	value="1.41421356237"	/>
-	<xacro:property name="phi4"    	value="0.785398163397"	/>
-	<xacro:property name="a4"    	value="0"	/>
-	<xacro:property name="alpha4"	value="${-pi/2}"	/>
-	<xacro:property name="d5"    	value="2"	/>
-	<xacro:property name="L5"    	value="2.0"	/>
-	<xacro:property name="phi5"    	value="0.0"	/>
+	<xacro:property name="L2"    	value="2.2360679775"	/>
+	<xacro:property name="phi2"    	value="0.463647609001"	/>
+	<xacro:property name="type1"    	value="revolute"	/>
+	<xacro:property name="a2"    	value="2"	/>
+	<xacro:property name="alpha2"	value="${3.14}"	/>
+	<xacro:property name="d3"    	value="0"	/>
+	<xacro:property name="L3"    	value="2.0"	/>
+	<xacro:property name="phi3"    	value="1.57079632679"	/>
+	<xacro:property name="type2"    	value="prismatic"	/>
 </robot>

File: manipulator/urdf/manipulator_main.xacro (robot description, xacro)
@@ -7,17 +7,13 @@
 	<my_link_cylinder name="${l01}" origin_xyz="${a1/2} 0 ${d2/2}" origin_rpy="0 ${phi2} 0" radius="${R01}" length="${L2}"/>
 	<my_link_cylinder name="${l02}" origin_xyz="${a2/2} 0 ${d3/2}" origin_rpy="0 ${phi3} 0" radius="${R02}" length="${L3}"/>
-	<my_link_cylinder name="${l03}" origin_xyz="${a3/2} 0 ${d4/2}" origin_rpy="0 ${phi4} 0" radius="${R03}" length="${L4}"/>
-	<my_link_cylinder name="${l04}" origin_xyz="${a4/2} 0 ${d5/2}" origin_rpy="0 ${phi5} 0" radius="${R04}" length="${L5}"/>
-<my_joint name="${l00}__${l01}" type="revolute"
+	<my_link_box name="${l03}" origin_xyz="${gripper_height_half} 0 0" origin_rpy="0 0 0" size="${gripper_size} ${gripper_height}"/>
+<my_joint name="${l00}__${l01}" type="${type0}"
 origin_rpy="${alpha0} 0 0" origin_xyz="${a0} 0 ${d1}"
 parent = "${l00}" child = "${l01}"/>
-<my_joint name="${l01}__${l02}" type="revolute"
+<my_joint name="${l01}__${l02}" type="${type1}"
 origin_rpy="${alpha1} 0 0" origin_xyz="${a1} 0 ${d2}"
 parent = "${l01}" child = "${l02}"/>
-<my_joint name="${l02}__${l03}" type="revolute"
+<my_joint name="${l02}__${l03}" type="${type2}"
 origin_rpy="${alpha2} 0 0" origin_xyz="${a2} 0 ${d3}"
 parent = "${l02}" child = "${l03}"/>
-<my_joint name="${l03}__${l04}" type="revolute"
-origin_rpy="${alpha3} 0 0" origin_xyz="${a3} 0 ${d4}"
-parent = "${l03}" child = "${l04}"/>
 </robot>

File: manipulator/urdf/templates.xacro (robot description, xacro)
@@ -33,3 +33,12 @@
 		</joint>
 	</xacro:macro>
+	<xacro:macro name="gripper_joint" params="name type origin_rpy origin_xyz parent child">
+		<joint name="${name}" type="${type}">
+			<axis xyz="0 0 1"/>
+			<limit effort="${limit_effort}" lower="${gripper_limit_lower}" upper="${gripper_limit_upper}" velocity="${limit_velocity}"/>
+			<origin xyz = "${origin_xyz}" rpy="${origin_rpy}"/>
+			<parent link = "${parent}"/>
+			<child link = "${child}"/>
+		</joint>
+	</xacro:macro>
 </robot>
